File: kicad/voltage-blaster.kicad_pcb (KiCad board)
At the start: 2 copper layers, 95.2 x 24.1 mm, 6 parts, among them J1 Bus_ISA_8bit, U1 LM7905

Commit message: updates
Parts:
- U1: footprint Package_TO_SOT_THT:TO-220-3_Horizontal_TabDown -> Sebs:TO-220-3_Horizontal_TabDown
- moved D1 1.62 mm to (153.0, 50.2), turned to 270 degrees
- moved R1 1.15 mm to (146.7, 57.8)
Connections:
- net Net-(C1-Pad2) renamed -5V
- net Net-(C2-Pad2) renamed -12V
- J1 pad 11: (no net) -> Net-(J1-Pad11)
- J1 pad 12: (no net) -> Net-(J1-Pad12)
- J1 pad 13: (no net) -> Net-(J1-Pad13)
- J1 pad 14: (no net) -> Net-(J1-Pad14)
- J1 pad 15: (no net) -> Net-(J1-Pad15)
- J1 pad 16: (no net) -> Net-(J1-Pad16)
- J1 pad 17: (no net) -> Net-(J1-Pad17)
- J1 pad 18: (no net) -> Net-(J1-Pad18)
- J1 pad 19: (no net) -> Net-(J1-Pad19)
- J1 pad 2: (no net) -> Net-(J1-Pad2)
- J1 pad 20: (no net) -> Net-(J1-Pad20)
- J1 pad 21: (no net) -> Net-(J1-Pad21)
- J1 pad 22: (no net) -> Net-(J1-Pad22)
- J1 pad 23: (no net) -> Net-(J1-Pad23)
- J1 pad 24: (no net) -> Net-(J1-Pad24)
- J1 pad 25: (no net) -> Net-(J1-Pad25)
- J1 pad 26: (no net) -> Net-(J1-Pad26)
- J1 pad 27: (no net) -> Net-(J1-Pad27)
- J1 pad 28: (no net) -> Net-(J1-Pad28)
- J1 pad 29: (no net) -> Net-(J1-Pad29)
- J1 pad 3: (no net) -> Net-(J1-Pad3)
- J1 pad 30: (no net) -> Net-(J1-Pad30)
- J1 pad 32: (no net) -> Net-(J1-Pad32)
- J1 pad 33: (no net) -> Net-(J1-Pad33)
- J1 pad 34: (no net) -> Net-(J1-Pad34)
- J1 pad 35: (no net) -> Net-(J1-Pad35)
- J1 pad 36: (no net) -> Net-(J1-Pad36)
- J1 pad 37: (no net) -> Net-(J1-Pad37)
- J1 pad 38: (no net) -> Net-(J1-Pad38)
- J1 pad 39: (no net) -> Net-(J1-Pad39)
- J1 pad 4: (no net) -> Net-(J1-Pad4)
- J1 pad 40: (no net) -> Net-(J1-Pad40)
- J1 pad 41: (no net) -> Net-(J1-Pad41)
- J1 pad 42: (no net) -> Net-(J1-Pad42)
- J1 pad 43: (no net) -> Net-(J1-Pad43)
- J1 pad 44: (no net) -> Net-(J1-Pad44)
- J1 pad 45: (no net) -> Net-(J1-Pad45)
- J1 pad 46: (no net) -> Net-(J1-Pad46)
- J1 pad 47: (no net) -> Net-(J1-Pad47)
- J1 pad 48: (no net) -> Net-(J1-Pad48)
- J1 pad 49: (no net) -> Net-(J1-Pad49)
- J1 pad 50: (no net) -> Net-(J1-Pad50)
- J1 pad 51: (no net) -> Net-(J1-Pad51)
- J1 pad 52: (no net) -> Net-(J1-Pad52)
- J1 pad 53: (no net) -> Net-(J1-Pad53)
- J1 pad 54: (no net) -> Net-(J1-Pad54)
- J1 pad 55: (no net) -> Net-(J1-Pad55)
- J1 pad 56: (no net) -> Net-(J1-Pad56)
- J1 pad 57: (no net) -> Net-(J1-Pad57)
- J1 pad 58: (no net) -> Net-(J1-Pad58)
- J1 pad 59: (no net) -> Net-(J1-Pad59)
- J1 pad 6: (no net) -> Net-(J1-Pad6)
- J1 pad 60: (no net) -> Net-(J1-Pad60)
- J1 pad 61: (no net) -> Net-(J1-Pad61)
- J1 pad 62: (no net) -> Net-(J1-Pad62)
- J1 pad 8: (no net) -> Net-(J1-Pad8)
- J1 pad 9: (no net) -> Net-(J1-Pad9)
Routing:
- net -12V: track 18.7 -> 28.7 mm
- net Net-(D1-Pad1): track 5.08 -> 6.98 mm
- net -5V: track 25.0 -> 26.1 mm
- net GND: track 16.1 -> 16.8 mm, vias 0 -> 1
- net (no net): vias 0 -> 82
Other:
- outline, holes or cut-outs redrawn
- board text added: "10"
- board text added: "31"
- board text added: "32"
- board text added: "5"
- board text added: "62"
- board text added: "7"
- board text added: "<- PC Rear"
- board text added: "HEATSINK"
- board text added: "PC Rear ->"
- board text added: "by PhilsComputerLab and Necroware"
- board text added: "rev 1.0.mod-hegars"
- board text removed: "PC back ----->"
- board text removed: "PC back <-----"
- board text removed: "by PhilsComputerLab & Necroware"
- board text removed: "rev 1.0"
