File: kicad/voltage-blaster-smd.kicad_pcb (KiCad board)
At the start: 2 copper layers, 95.2 x 24.1 mm, 14 parts, among them J1 Bus_ISA_8bit, U1 LM7905

Commit message: Update voltage-blaster-smd.kicad_pcb
Parts:
- moved F2 0.25 mm to (141.6, 58.7)
- moved F1 0.13 mm to (146.7, 58.7)
Routing:
- net -12V: track 36.6 -> 57.6 mm, vias 0 -> 2
- net -5V: track 36.5 -> 42.9 mm, vias 1 -> 3
- net GND: track 28.7 -> 29.5 mm
- net Net-(F2-Pad1): vias 1 -> 0
- net Net-(F1-Pad1): vias 1 -> 0
Other:
- board text added: "-12v"
- board text added: "-5v"
- board text added: "GND"
- board text added: "Original design concept by PhilsComputerLab and Necroware"
- board text added: "https://pcb.hegars.com/?sku=vbsmd2?sn="
- board text added: "ver 2.0.smd"
- board text removed: "by PhilsComputerLab and Necroware"
- board text removed: "rev 2.0.smd.mod-hegars"
Changed lines of the file:
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@@
   (general
     (thickness 1.6)
-    (drawings 57)
-    (tracks 33)
+    (drawings 62)
+    (tracks 41)
     (zones 0)
     (modules 14)
@@
     (37 F.SilkS user)
     (38 B.Mask user)
-    (39 F.Mask user hide)
+    (39 F.Mask user)
     (40 Dwgs.User user)
     (41 Cmts.User user)
@@
   )
   (module Fuse_Holders_and_Fuses:Fuse_SMD1206_HandSoldering (layer F.Cu)
-    (at 141.605 58.928 90)
+    (at 141.605 58.674 90)
     (descr "Fuse, Sicherung, SMD1206, Littlefuse-Wickmann 433 Series, Hand Soldering,")
     (tags "Fuse Sicherung SMD1206 Littlefuse-Wickmann 433 Series Hand Soldering ")
@@
     (pad 2 smd rect (at 2.09 0 180) (size 2.03 2.65) (layers F.Cu F.Paste F.Mask)
       (net 4 -12V))
+    (model ${KISYS3DMOD}/Fuse.3dshapes/Fuse_1206_3216Metric.wrl
+      (at (xyz 0 0 0))
+      (scale (xyz 1 1 1))
+      (rotate (xyz 0 0 0))
+    )
   )
   (module Fuse_Holders_and_Fuses:Fuse_SMD1206_HandSoldering (layer F.Cu)
-    (at 146.685 58.801 90)
+    (at 146.685 58.674 90)
     (descr "Fuse, Sicherung, SMD1206, Littlefuse-Wickmann 433 Series, Hand Soldering,")
     (tags "Fuse Sicherung SMD1206 Littlefuse-Wickmann 433 Series Hand Soldering ")
@@
     (pad 2 smd rect (at 2.09 0 180) (size 2.03 2.65) (layers F.Cu F.Paste F.Mask)
       (net 3 -5V))
+    (model ${KISYS3DMOD}/Fuse.3dshapes/Fuse_1206_3216Metric.wrl
+      (at (xyz 0 0 0))
+      (scale (xyz 1 1 1))
+      (rotate (xyz 0 0 0))
+    )
   )
   (module TO_SOT_Packages_SMD:TO-263-3_TabPin2 (layer F.Cu)
@@
       (rotate (xyz 0 0 0))
     )
+    (model ${KISYS3DMOD}/TO_SOT_Packages_SMD.3dshapes/TO-263-3Lead.wrl
+      (offset (xyz -6 0 0))
+      (scale (xyz 1 1 1))
+      (rotate (xyz 0 0 90))
+    )
   )
   (module Measurement_Points:Measurement_Point_Round-SMD-Pad_Big (layer B.Cu)
@@
     (tags "Mesurement Point Round SMD Pad 3mm")
     (attr virtual)
-    (fp_text reference TP3 (at 0 3) (layer B.SilkS)
+    (fp_text reference TP3 (at 0 3) (layer B.SilkS) hide
       (effects (font (size 1 1) (thickness 0.15)) (justify mirror))
     )
@@
     (tags "Mesurement Point Round SMD Pad 3mm")
     (attr virtual)
-    (fp_text reference TP2 (at 0 3) (layer B.SilkS)
+    (fp_text reference TP2 (at 0 3) (layer B.SilkS) hide
       (effects (font (size 1 1) (thickness 0.15)) (justify mirror))
     )
@@
     (tags "Mesurement Point Round SMD Pad 3mm")
     (attr virtual)
-    (fp_text reference TP1 (at 0 3) (layer B.SilkS)
+    (fp_text reference TP1 (at 0 3) (layer B.SilkS) hide
       (effects (font (size 1 1) (thickness 0.15)) (justify mirror))
     )
@@
     (tags "mounting hole 2.5mm")
     (attr virtual)
-    (fp_text reference H1 (at 0 -3.5) (layer F.SilkS)
+    (fp_text reference H1 (at 0 -3.5) (layer F.SilkS) hide
       (effects (font (size 1 1) (thickness 0.15)))
     )
@@
       (net 1 GND))
   )
+  (gr_text -12v (at 141.732 54.102) (layer B.SilkS)
+    (effects (font (size 1 1) (thickness 0.15)) (justify mirror))
+  )
+  (gr_text -5v (at 146.939 54.102) (layer B.SilkS)
+    (effects (font (size 1 1) (thickness 0.15)) (justify mirror))
+  )
+  (gr_text GND (at 156.845 54.102) (layer B.SilkS)
+    (effects (font (size 1 1) (thickness 0.15)) (justify mirror))
+  )
+  (gr_poly (pts (xy 89.535 60.579) (xy 72.39 60.579) (xy 72.39 57.277) (xy 89.535 57.277)) (layer B.SilkS) (width 0.1))
+  (gr_text https://pcb.hegars.com/?sku=vbsmd2?sn= (at 114.681 58.801) (layer B.SilkS)
+    (effects (font (size 1.5 1.5) (thickness 0.2)) (justify mirror))
+  )
+  (gr_text "Voltage\nBlaster\nSMD" (at 83.185 53.975) (layer F.Mask)
+    (effects (font (size 2 2) (thickness 0.3)) (justify left))
+  )
   (gr_line (start 159.639 49.022) (end 138.557 49.022) (layer B.SilkS) (width 0.12))
   (gr_line (start 159.639 55.499) (end 159.639 49.022) (layer B.SilkS) (width 0.12))
   (gr_line (start 138.557 55.499) (end 159.639 55.499) (layer B.SilkS) (width 0.12))
   (gr_line (start 138.557 49.022) (end 138.557 55.499) (layer B.SilkS) (width 0.12))
-  (gr_poly (pts (xy 112.268 61.722) (xy 82.423 61.722) (xy 82.423 48.514) (xy 112.268 48.514)) (layer F.Cu) (width 0.1))
-  (gr_text "TEST \nPOINTS" (at 151.892 51.562) (layer B.SilkS)
+  (gr_poly (pts (xy 112.268 61.5315) (xy 82.423 61.5315) (xy 82.423 48.514) (xy 112.268 48.514)) (layer F.Cu) (width 0.1))
+  (gr_text "TEST \nPOINTS" (at 151.892 52.578) (layer B.SilkS)
     (effects (font (size 1 1) (thickness 0.15)) (justify mirror))
   )
@@
   (gr_line (start 163.957 58.547) (end 163.957 60.452) (layer F.SilkS) (width 0.12))
   (gr_arc (start 77.47 53.34) (end 77.47 46.99) (angle -90) (layer Edge.Cuts) (width 0.05))
-  (gr_text "Voltage Blaster SMD" (at 112.014 52.07) (layer B.Mask)
-    (effects (font (size 3 3) (thickness 0.5)) (justify mirror))
-  )
   (gr_arc (start 160.02 53.34) (end 166.37 53.34) (angle -90) (layer Edge.Cuts) (width 0.05))
   (gr_text 1 (at 156.845 62.23) (layer B.SilkS)
     (effects (font (size 1 1) (thickness 0.15)) (justify mirror))
   )
-  (gr_text "rev 2.0.smd.mod-hegars" (at 97.282 61.214) (layer B.SilkS)
-    (effects (font (size 1.2 1.2) (thickness 0.15)) (justify mirror))
-  )
-  (gr_text "by PhilsComputerLab \nand Necroware" (at 103.886 57.15) (layer F.Fab)
-    (effects (font (size 1.8 1.5) (thickness 0.2)) (justify mirror))
+  (gr_text "ver 2.0.smd" (at 90.17 60.198) (layer F.SilkS)
+    (effects (font (size 1.2 1.2) (thickness 0.15)))
+  )
+  (gr_text "Original design concept by \nPhilsComputerLab and Necroware" (at 109.474 52.07) (layer B.SilkS)
+    (effects (font (size 1 1) (thickness 0.15)) (justify left mirror))
   )
   (gr_text 32 (at 156.845 62.23) (layer F.SilkS)
@@
   (gr_line (start 166.37 63.5) (end 166.37 53.34) (layer Edge.Cuts) (width 0.05))
   (gr_line (start 158.75 63.5) (end 166.37 63.5) (layer Edge.Cuts) (width 0.05))
-  (via (at 141.605 60.96) (size 0.8) (drill 0.4) (layers F.Cu B.Cu) (net 7))
-  (via (at 146.685 60.96) (size 0.8) (drill 0.4) (layers F.Cu B.Cu) (net 6))
-  (via (at 80.645 60.96) (size 0.8) (drill 0.4) (layers F.Cu B.Cu) (net 1))
-  (via (at 133.985 60.96) (size 0.8) (drill 0.4) (layers F.Cu B.Cu) (net 1))
+  (via (at 141.605 60.579) (size 0.8) (drill 0.4) (layers F.Cu B.Cu) (net 4))
+  (via (at 146.685 60.579) (size 0.8) (drill 0.4) (layers F.Cu B.Cu) (net 3))
+  (via (at 80.645 60.579) (size 0.8) (drill 0.4) (layers F.Cu B.Cu) (net 1))
+  (via (at 133.985 60.579) (size 0.8) (drill 0.4) (layers F.Cu B.Cu) (net 1))
   (via (at 146.685 51.562) (size 0.8) (drill 0.4) (layers F.Cu B.Cu) (net 3))
-  (via (at 156.845 60.96) (size 0.8) (drill 0.4) (layers F.Cu B.Cu) (net 1))
-  (segment (start 156.845 67.31) (end 156.845 60.96) (width 0.5) (layer B.Cu) (net 1))
-  (segment (start 156.845 60.96) (end 156.845 51.308) (width 0.5) (layer B.Cu) (net 1))
-  (segment (start 80.645 67.31) (end 80.645 60.96) (width 0.5) (layer B.Cu) (net 1))
-  (segment (start 133.985 67.31) (end 133.985 60.96) (width 0.5) (layer B.Cu) (net 1))
+  (via (at 156.845 60.579) (size 0.8) (drill 0.4) (layers F.Cu B.Cu) (net 1))
+  (segment (start 156.845 60.579) (end 156.845 67.31) (width 0.5) (layer B.Cu) (net 1))
+  (segment (start 156.845 60.579) (end 156.845 51.308) (width 0.5) (layer B.Cu) (net 1))
+  (segment (start 133.985 60.579) (end 133.985 67.31) (width 0.5) (layer B.Cu) (net 1))
+  (segment (start 80.645 60.579) (end 80.645 67.31) (width 0.5) (layer B.Cu) (net 1))
   (segment (start 153.13 49.53) (end 157.004 49.53) (width 0.5) (layer F.Cu) (net 2))
   (segment (start 121.5228 52.4764) (end 125.2474 52.4764) (width 0.5) (layer F.Cu) (net 3))
@@
   (segment (start 148.209 51.562) (end 149.13 50.641) (width 0.5) (layer F.Cu) (net 3))
   (segment (start 146.685 51.562) (end 148.209 51.562) (width 0.5) (layer F.Cu) (net 3))
-  (segment (start 146.685 56.711) (end 146.685 51.562) (width 0.5) (layer F.Cu) (net 3))
+  (segment (start 146.685 56.711) (end 146.685 56.711) (width 0.5) (layer F.Cu) (net 3))
+  (via (at 146.685 56.388) (size 0.8) (drill 0.4) (layers F.Cu B.Cu) (net 3))
+  (segment (start 146.685 60.579) (end 146.685 67.31) (width 0.5) (layer B.Cu) (net 3))
+  (segment (start 146.685 56.388) (end 146.685 51.562) (width 0.5) (layer B.Cu) (net 3))
   (segment (start 141.565 67.27) (end 141.605 67.31) (width 0.5) (layer B.Cu) (net 4))
   (segment (start 135.288 56.675) (end 135.288 58.674) (width 0.5) (layer F.Cu) (net 4))
@@
   (segment (start 149.13 58.007) (end 149.13 53.848) (width 0.5) (layer F.Cu) (net 4))
   (segment (start 148.463 58.674) (end 149.13 58.007) (width 0.5) (layer F.Cu) (net 4))
+  (segment (start 141.605 56.838) (end 141.605 56.838) (width 0.5) (layer F.Cu) (net 4))
   (segment (start 141.605 56.838) (end 141.605 58.674) (width 0.5) (layer F.Cu) (net 4))
+  (via (at 141.605 56.515) (size 0.8) (drill 0.4) (layers F.Cu B.Cu) (net 4))
+  (segment (start 141.605 60.579) (end 141.605 67.31) (width 0.5) (layer B.Cu) (net 4))
+  (segment (start 141.605 56.515) (end 141.605 51.435) (width 0.5) (layer B.Cu) (net 4))
+  (segment (start 121.5228 55.0164) (end 112.3728 55.0164) (width 0.5) (layer F.Cu) (net 4))
   (segment (start 153.13 53.848) (end 157.004 53.848) (width 0.5) (layer F.Cu) (net 5))
   (zone (net 1) (net_name GND) (layer B.Cu) (hatch edge 0.508)
-    (connect_pads thru_hole_only (clearance 0.508))
+    (connect_pads yes (clearance 0.508))
     (min_thickness 0.254)
     (fill yes (arc_segments 32) (thermal_gap 0.508) (thermal_bridge_width 0.508))
@@
   )
   (zone (net 1) (net_name GND) (layer F.Cu) (hatch edge 0.508)
-    (connect_pads thru_hole_only (clearance 0.508))
+    (connect_pads yes (clearance 0.508))
     (min_thickness 0.254)
     (fill yes (arc_segments 32) (thermal_gap 0.508) (thermal_bridge_width 0.508))
