File: kicad/voltage-blaster-smd.kicad_pcb (KiCad board)
At the start: 2 copper layers, 95.2 x 24.1 mm, 14 parts, among them J1 Bus_ISA_8bit, U1 LM7905

Commit message: updates
Other:
- board text added: "https://pcb.hegars.com/?sku=vbsmd2&sn="
- board text removed: "https://pcb.hegars.com/?sku=vbsmd2?sn="
